File: PCB/main.kicad_sch (KiCad schematic)
At the start: 0 parts

Commit message: update mobile-test-stand-tryout,
Parts:
- added D1, D2, D3, D4, D5: LED, Diode_SMD:D_0805_2012Metric, symbol Device:LED
- added H1, H2, H3, H4: MountingHole, MountingHole:MountingHole_3.2mm_M3_ISO14580, symbol Mechanical:MountingHole
- added J1: ATX-24, Connector_Molex:Molex_Mini-Fit_Jr_5569-24A2_2x12_P4.20mm_Horizontal, symbol Connector:ATX-24
- added J2: Conn_RPi, Connector_PinHeader_2.54mm:PinHeader_1x04_P2.54mm_Horizontal, symbol Connector:Conn_01x04_Male
- added J3: Conn_USB_HUBS, Connector_PinHeader_2.54mm:PinHeader_1x04_P2.54mm_Horizontal, symbol Connector:Conn_01x04_Male
- added J4: Conn_Router, Connector_PinHeader_2.54mm:PinHeader_1x04_P2.54mm_Horizontal, symbol Connector:Conn_01x04_Male
- added J5: Conn_MOBILE, Connector_PinHeader_2.54mm:PinHeader_1x04_P2.54mm_Horizontal, symbol Connector:Conn_01x04_Male
- added J6: Conn_NUC, Connector_PinHeader_2.54mm:PinHeader_1x04_P2.54mm_Horizontal, symbol Connector:Conn_01x04_Male
- added R1: R331, Resistor_SMD:R_0805_2012Metric, symbol Device:R
- added R2, R3: R221, Resistor_SMD:R_0805_2012Metric, symbol Device:R
- added R4, R5: R102, Resistor_SMD:R_0805_2012Metric, symbol Device:R
Connections:
- new net: D5.1 (K), R5.1
- new net: D3.1 (K), R3.1
- new net: D1.1 (K), R1.1
- new net: D2.1 (K), R2.1
- new net: D4.1 (K), R4.1
- new net -12V: J1.14 (-12V)
- new net 12V: D1.2 (A), J1.10 (+12V), J1.11 (+12V), J3.1 (Pin_1), J4.1 (Pin_1), J5.1 (Pin_1), J6.1 (Pin_1)
- new net 3V3: D4.2 (A), J1.1 (+3.3V), J1.12 (+3.3V), J1.13 (+3.3V), J1.2 (+3.3V), J3.3 (Pin_3), J4.3 (Pin_3), J5.3 (Pin_3), J6.3 (Pin_3)
- new net 5V: D2.2 (A), J1.21 (+5V), J1.22 (+5V), J1.23 (+5V), J1.4 (+5V), J1.6 (+5V), J3.2 (Pin_2), J4.2 (Pin_2), J5.2 (Pin_2), J6.2 (Pin_2)
- new net 5V_SB: D3.2 (A), J1.9 (+5VSB), J2.1 (Pin_1)
- new net GND: J1.15 (GND), J1.17 (GND), J1.18 (GND), J1.19 (GND), J1.24 (GND), J1.3 (GND), J1.5 (GND), J1.7 (GND), J2.4 (Pin_4), J3.4 (Pin_4), J4.4 (Pin_4), J5.4 (Pin_4), J6.4 (Pin_4), R1.2, R2.2, R3.2, R4.2, R5.2
- new net PS_ON: D5.2 (A), J1.16 (PS_ON#), J2.2 (Pin_2)
- new net PWR_OK: J1.8 (PWR_OK), J2.3 (Pin_3)
