File: PCB/main.kicad_pcb (KiCad board)
At the start: 2 copper layers, 0 parts

Commit message: update mobile-test-stand-tryout,
Parts:
- added D1: LED, Diode_SMD:D_0805_2012Metric, F.Cu at (54.5, 30.0)
- added D2: LED, Diode_SMD:D_0805_2012Metric, F.Cu at (54.5, 34.5)
- added D3: LED, Diode_SMD:D_0805_2012Metric, F.Cu at (54.5, 39.5)
- added D4: LED, Diode_SMD:D_0805_2012Metric, F.Cu at (54.5, 44.5)
- added D5: LED, Diode_SMD:D_0805_2012Metric, F.Cu at (54.5, 49.5)
- added H1: MountingHole, MountingHole:MountingHole_3.2mm_M3_ISO14580, F.Cu at (30.0, 30.0)
- added H2: MountingHole, MountingHole:MountingHole_3.2mm_M3_ISO14580, F.Cu at (110.0, 30.0)
- added H3: MountingHole, MountingHole:MountingHole_3.2mm_M3_ISO14580, F.Cu at (30.0, 110.0)
- added H4: MountingHole, MountingHole:MountingHole_3.2mm_M3_ISO14580, F.Cu at (110.0, 110.0)
- added J1: ATX-24, Connector_Molex:Molex_Mini-Fit_Jr_5569-24A2_2x12_P4.20mm_Horizontal, F.Cu at (40.3, 84.1)
- added J2: Conn_RPi, Connector_PinHeader_2.54mm:PinHeader_1x04_P2.54mm_Horizontal, F.Cu at (99.3, 103.1)
- added J3: Conn_USB_HUBS, Connector_PinHeader_2.54mm:PinHeader_1x04_P2.54mm_Horizontal, F.Cu at (74.3, 103.1)
- added J4: Conn_Router, Connector_PinHeader_2.54mm:PinHeader_1x04_P2.54mm_Horizontal, F.Cu at (60.8, 103.1)
- added J5: Conn_MOBILE, Connector_PinHeader_2.54mm:PinHeader_1x04_P2.54mm_Horizontal, F.Cu at (86.5, 103.1)
- added J6: Conn_NUC, Connector_PinHeader_2.54mm:PinHeader_1x04_P2.54mm_Horizontal, F.Cu at (47.3, 103.1)
- added R1: R331, Resistor_SMD:R_0805_2012Metric, F.Cu at (61.0, 30.0)
- added R2: R221, Resistor_SMD:R_0805_2012Metric, F.Cu at (61.0, 34.5)
- added R3: R221, Resistor_SMD:R_0805_2012Metric, F.Cu at (61.0, 39.5)
- added R4: R102, Resistor_SMD:R_0805_2012Metric, F.Cu at (60.9, 44.5)
- added R5: R102, Resistor_SMD:R_0805_2012Metric, F.Cu at (61.0, 49.5)
Routing:
- net /5V_SB: track 0.00 -> 219.9 mm, vias 0 -> 1
- net /12V: track 0.00 -> 200.1 mm
- net GND: track 0.00 -> 198.8 mm
- net /5V: track 0.00 -> 168.7 mm, vias 0 -> 1
- net /3V3: track 0.00 -> 165.4 mm, vias 0 -> 1
- net /PWR_OK: track 0.00 -> 121.4 mm
- net /PS_ON: track 0.00 -> 86.5 mm, vias 0 -> 1
- net Net-(D3-Pad1): track 0.00 -> 8.98 mm, vias 0 -> 2
- net Net-(D1-Pad1): track 0.00 -> 8.73 mm
- net Net-(D4-Pad1): track 0.00 -> 8.40 mm
- net Net-(D5-Pad1): track 0.00 -> 8.26 mm
- net Net-(D2-Pad1): track 0.00 -> 6.65 mm, vias 0 -> 2
Other:
- board outline added: 90 x 90 mm
- board text added: "Louislabs ATX-power distribution board louiscklaw.github.io"

Commit message: update before fabrication,
Parts:
- added FID1: Fiducial, Fiducial:Fiducial_1mm_Mask3mm, F.Cu at (82.0, 32.0)
- added FID2: Fiducial, Fiducial:Fiducial_1.5mm_Mask3mm, F.Cu at (112.0, 104.0)
- added FID3: Fiducial, Fiducial:Fiducial_0.75mm_Mask2.25mm, F.Cu at (35.0, 110.0)
- added J10: Conn_USB_HUBS, Connector_PinHeader_2.54mm:PinHeader_1x04_P2.54mm_Horizontal, F.Cu at (103.5, 78.0)
- added J11: Conn_USB_HUBS, Connector_PinHeader_2.54mm:PinHeader_1x04_P2.54mm_Horizontal, F.Cu at (103.5, 91.0)
- added J12: POWER_ON, Connector_PinHeader_2.54mm:PinHeader_1x02_P2.54mm_Vertical, F.Cu at (82.0, 37.0)
- added J7: Conn_USB_HUBS, Connector_PinHeader_2.54mm:PinHeader_1x04_P2.54mm_Horizontal, F.Cu at (103.0, 37.5)
- added J8: Conn_USB_HUBS, Connector_PinHeader_2.54mm:PinHeader_1x04_P2.54mm_Horizontal, F.Cu at (103.1, 51.2)
- added J9: Conn_USB_HUBS, Connector_PinHeader_2.54mm:PinHeader_1x04_P2.54mm_Horizontal, F.Cu at (103.5, 64.5)
- added TP1: TestPoint, Connector_PinHeader_2.54mm:PinHeader_1x01_P2.54mm_Vertical, F.Cu at (93.0, 30.7)
- added TP2: TestPoint, Connector_PinHeader_2.54mm:PinHeader_1x01_P2.54mm_Vertical, F.Cu at (88.3, 35.4)
- added TP3: TestPoint, Connector_PinHeader_2.54mm:PinHeader_1x01_P2.54mm_Vertical, F.Cu at (93.0, 44.6)
- added TP4: TestPoint, Connector_PinHeader_2.54mm:PinHeader_1x01_P2.54mm_Vertical, F.Cu at (93.0, 40.0)
- added TP5: TestPoint, Connector_PinHeader_2.54mm:PinHeader_1x01_P2.54mm_Vertical, F.Cu at (88.3, 30.7)
- added TP6: TestPoint, Connector_PinHeader_2.54mm:PinHeader_1x01_P2.54mm_Vertical, F.Cu at (88.3, 44.6)
- added TP7: TestPoint, Connector_PinHeader_2.54mm:PinHeader_1x01_P2.54mm_Vertical, F.Cu at (88.3, 40.0)
- added TP8: TestPoint, Connector_PinHeader_2.54mm:PinHeader_1x01_P2.54mm_Vertical, F.Cu at (93.0, 35.4)
Routing:
- net /3V3: track 165.4 -> 512.1 mm, vias 1 -> 4
- net GND: track 198.8 -> 503.7 mm, vias 0 -> 15
- net /12V: track 200.1 -> 440.0 mm, vias 0 -> 3
- net /5V: track 168.7 -> 374.5 mm, vias 1 -> 4
- net /-12V: track 0.00 -> 83.0 mm, vias 0 -> 3
- net /PS_ON: track 86.5 -> 155.6 mm, vias 1 -> 2
- net /5V_SB: track 219.9 -> 168.1 mm
- net /PWR_OK: track 121.4 -> 166.3 mm, vias 0 -> 1
- net Net-(D4-Pad1): track 8.40 -> 17.7 mm, vias 0 -> 2
- net Net-(D2-Pad1): track 6.65 -> 8.80 mm, vias 2 -> 0
- net Net-(D1-Pad1): track 8.73 -> 10.3 mm
- net Net-(D5-Pad1): track 8.26 -> 9.67 mm
- net Net-(D3-Pad1): track 8.98 -> 9.34 mm, vias 2 -> 0
Other:
- board text added: "12V HEALTHY"
- board text added: "3V3 HEALTHY"
- board text added: "5V HEALTHY"
- board text added: "5V_SB HEALTHY"
- board text added: "CHECKLIST 1. show board dimensions 1. SILKSCREEN 1. TRACKS 1. VIAS 1. FIDUCIO 1. MECHANICAL / MOUNTINGS 1. FOOTPRINTS 1. Test points"
- board text added: "Fabrication option: green pcb 1oz 1.6 FR-4"
- board text added: "PS_ON"

Commit message: update mobile-test-stand-tryout,
Other:
- board text added: "TODO (REV 1): 1. move green terminal nearer to board edge"
Changed lines of the file:
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@@
+    (effects (font (size 1.5 1.5) (thickness 0.3)) (justify left))
+  )
+  (gr_text "TODO (REV 1):\n\n1. move green terminal nearer to board edge" (at 194 25) (layer "B.Cu")
     (effects (font (size 1.5 1.5) (thickness 0.3)) (justify left))
   )

Commit message: update mobile-test-stand-tryout,
Other:
- board text added: "TODO (REV 1): 1. move green terminal nearer to board edge 2. make testpoints to 2.54 headers"
- board text removed: "TODO (REV 1): 1. move green terminal nearer to board edge"
Changed lines of the file:
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@@
     (effects (font (size 1.5 1.5) (thickness 0.3)) (justify left))
   )
-  (gr_text "TODO (REV 1):\n\n1. move green terminal nearer to board edge" (at 194 25) (layer "B.Cu")
+  (gr_text "TODO (REV 1):\n\n1. move green terminal nearer to board edge\n2. make testpoints to 2.54 headers" (at 194 25) (layer "B.Cu")
     (effects (font (size 1.5 1.5) (thickness 0.3)) (justify left))
   )
